File: RVario6/main.brd (EAGLE design)
At the start: 160 x 100 mm, 7 parts, among them J1 ZX62-B-5PA, U1 32U4

Commit message: Finished schematic RVario6
Parts:
- added C10, C11, C14, C6, C7, C8, C9: 100nf, Seeed-Capacitor:C0603
- added C12: 10nf, Seeed-Capacitor:C0603
- added C13: 1uf, Seeed-Capacitor:C0603
- added C15, C3, C4, C5: 10uf, Seeed-Capacitor:C0805
- added D1, D2: 40V-500MA, Seeed-Diode:SOD-123
- added D3: GREEN-0603, Seeed-LED:LED-0603
- added D4: BLUE-0603, Seeed-LED:LED-0603
- added IC1: BMP280, bosch-bmp280:BMP280
- added IC2: W25Q32BVWSON8_6X5, Custom_old:SON127P600X500X75-8
- added J2: 2x3p-2.54, Seeed-Connector:H2X3-2.54
- added J3: 455-1750-1-ND, SparkFun-Connectors:1X03
- added J4: I2C1, SparkFun-Connectors:1X04
- added J5: I2C2, SparkFun-Connectors:1X04
- added J6: GPS, SparkFun-Connectors:1X04
- added K1: (no value), Seeed-Switch:SW4-SMD-6.0X6.0X5.0MM
- added R3, R4, R7, R8: 2.2K, Seeed-Resistor:R0603
- added R5, R6: 220R, Seeed-Resistor:R0603
- added U$1, U$2: PADPAD_2.5X1.5, Custom_old:PAD_2.5X1.5
- added U$3, U$4: MS5611, Custom_old:MS5611
- added U$5: MS5637, Custom_old:MS5637
- added U$6, U$7: MS5525, Custom_old:SOIC14-WIDE
- added U2: 433MHz, SparkFun-RF:RFM69HCW-XXXS2
- added U3: CJT1117-3.3-SOT223, Seeed-IC:SOT-223
- added U4: (no value), Seeed-Sensor:QFN24G-0.4-3X3MM
- C1, C2: value 10pF -> 10uf; device SparkFun-Capacitors:0603 -> Seeed-Capacitor:C0805
- Y1: value (none) -> 8MHZ; device SparkFun-Clocks:CRYSTAL-SMD-5X3.2-4PAD -> Seeed-Crystal Oscillator:X3-SMD-3.6X1.3X0.8MM
- moved C2 48.7 mm to (-38.1, -53.3)
- moved C1 47.5 mm to (-38.1, -48.3)
- moved Y1 36.9 mm to (-33.0, -19.1)
- moved R1 24.1 mm to (2.00, 19.0)
Connections:
- new net CS_5525_1: U$6.8
- new net CS_5525_2: U$7.8
- new net CS_5611_1: U$3.4, U$3.5, U1.38
- new net CS_5611_2: U$4.4, U$4.5, U1.37
- new net CS_BMP: IC1.2
- new net CS_RFM: U1.8, U2.5
- new net LED_B: R6.1
- new net LED_G: R5.1
- new net MISO: IC1.5, U$3.6, U$4.6, U$6.5, U$7.5, U1.11, U2.2
- new net MOSI: IC1.3, U$3.7, U$4.7, U$6.6, U$7.6, U1.10, U2.3
- new net N$10: C11.2, U4.10
- new net N$11: U$7.1, U$7.3
- new net N$12: U$7.2, U$7.4
- new net N$13: U$7.12, U$7.14
- new net N$14: D3.+, R5.2
- new net N$15: D4.+, R6.2
- new net N$16: C13.2, U1.6
- new net N$17: J3.3, R7.2
- new net N$18: R8.1, U1.13
- new net N$19: C14.2, U1.42
- new net N$5: C1.2, D1.-, D2.-, U3.3
- new net N$6: U$2.1, U2.9
- new net N$7: U$6.1, U$6.3
- new net N$8: U$6.2, U$6.4
- new net N$9: U$6.12, U$6.14
- new net RC_IN: R7.1
- new net RFM_D0: U1.32, U2.14
- new net RFM_D1: U2.15
- new net RFM_D2: U2.16
- new net SCK: IC1.4, U$3.8, U$4.8, U$6.7, U$7.7, U1.9, U2.4
- new net SCL: R3.1, U$5.3, U1.18, U4.23
- new net SDA: R4.1, U$5.2, U1.19, U4.24
- new net VCC: C10.2, C12.2, C2.2, C3.2, C4.2, C5.2, C6.2, C7.2, C8.2, C9.2, IC1.6, IC1.8, R3.2, R4.2, R8.2, U$3.1, U$4.1, U$5.1, U$6.11, U$6.13, U$7.11, U$7.13, U1.14, U1.24, U1.34, U1.44, U2.13, U3.2, U3.TER, U4.1, U4.13, U4.22, U4.8
- new net V_RC: D1.+, J3.2
- new net V_USB: C15.2, D2.+, J1.1, U1.2, U1.7
- net GND: now also C10.1, C11.1, C12.1, C13.1, C14.1, C15.1, C2.1, C3.1, C4.1, C5.1, C6.1, C7.1, C8.1, C9.1, D3.-, D4.-, IC1.1, IC1.7, J3.1, U$1.1, U$3.2, U$3.3, U$4.2, U$4.3, U$5.4, U$6.10, U$6.9, U$7.10, U$7.9, U2.1, U2.10, U2.8, U3.1, U4.18, U4.20, U4.9, Y1.2; no longer C2.2
- net N$1: now also Y1.1; no longer C1.2, Y1.3
- net N$2: now also Y1.3; no longer C2.1, Y1.1
Other:
- board size 160 x 100 mm -> 47 x 31 mm

Commit message: Rvario6 updates
Parts:
- added J7: MICROSD-9P, Seeed-Connector:MICRO-SD9+4P-SMD-16.1X14.5X1.85MM
Other:
- board size 47 x 31 mm -> 61 x 34 mm
Changed lines of the file:
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@@
 <board>
 <plain>
-<wire x1="0" y1="0" x2="47" y2="0" width="0" layer="20"/>
-<wire x1="47" y1="0" x2="47" y2="31" width="0" layer="20"/>
-<wire x1="47" y1="31" x2="0" y2="31" width="0" layer="20"/>
-<wire x1="0" y1="31" x2="0" y2="0" width="0" layer="20"/>
+<wire x1="0" y1="0" x2="61" y2="0" width="0" layer="20"/>
+<wire x1="61" y1="0" x2="61" y2="34" width="0" layer="20"/>
+<wire x1="61" y1="34" x2="0" y2="34" width="0" layer="20"/>
+<wire x1="0" y1="34" x2="0" y2="0" width="0" layer="20"/>
 </plain>
 <attributes>
@@
 <attribute name="MPN" value="DTSM-62K-S-V-T/R(SN431)" x="-157" y="-209" size="1.778" layer="27" display="off"/>
 </element>
+<element name="J7" library="Seeed-Connector" package="MICRO-SD9+4P-SMD-16.1X14.5X1.85MM" value="MICROSD-9P" x="-182" y="-203"/>
 </elements>
 <signals>
@@
 <contactref element="R1" pad="2"/>
 <contactref element="U1" pad="3"/>
-<wire x1="2.85" y1="19" x2="-27.4665" y2="7.82886875" width="0" layer="19" extent="1-1"/>
+<wire x1="-27.4665" y1="7.82886875" x2="2.85" y2="19" width="0" layer="19" extent="1-1"/>
 </signal>
 <signal name="D+">
@@
 <contactref element="U$7" pad="5"/>
 <wire x1="-101.975" y1="-94.2" x2="-94.92" y2="-110" width="0" layer="19" extent="1-1"/>
-<wire x1="35.08" y1="20" x2="-101.975" y2="-94.2" width="0" layer="19" extent="1-1"/>
-<wire x1="-61.9" y1="-84.625" x2="35.08" y2="20" width="0" layer="19" extent="1-1"/>
+<wire x1="-61.9" y1="-84.625" x2="-101.975" y2="-94.2" width="0" layer="19" extent="1-1"/>
 <wire x1="-61.9" y1="-78.625" x2="-61.9" y2="-84.625" width="0" layer="19" extent="1-1"/>
 <wire x1="-27.4665" y1="3.892265625" x2="-61.9" y2="-78.625" width="0" layer="19" extent="1-1"/>
 <wire x1="20.5" y1="18" x2="-27.4665" y2="3.892265625" width="0" layer="19" extent="1-16"/>
+<wire x1="35.08" y1="20" x2="20.5" y2="18" width="0" layer="19" extent="1-16"/>
 </signal>
 <signal name="MOSI">
@@
 <contactref element="U$7" pad="6"/>
 <wire x1="-101.325" y1="-95.8" x2="-93.65" y2="-110" width="0" layer="19" extent="1-1"/>
-<wire x1="36.35" y1="20" x2="-101.325" y2="-95.8" width="0" layer="19" extent="1-1"/>
-<wire x1="-61.9" y1="-83.375" x2="36.35" y2="20" width="0" layer="19" extent="1-1"/>
+<wire x1="-61.9" y1="-83.375" x2="-101.325" y2="-95.8" width="0" layer="19" extent="1-1"/>
 <wire x1="-61.9" y1="-77.375" x2="-61.9" y2="-83.375" width="0" layer="19" extent="1-1"/>
 <wire x1="-27.4665" y1="4.392265625" x2="-61.9" y2="-77.375" width="0" layer="19" extent="1-1"/>
 <wire x1="20.5" y1="16" x2="-27.4665" y2="4.392265625" width="0" layer="19" extent="1-16"/>
+<wire x1="36.35" y1="20" x2="20.5" y2="16" width="0" layer="19" extent="1-16"/>
 </signal>
 <signal name="SCK">
@@
 <contactref element="U$7" pad="7"/>
 <wire x1="-101.975" y1="-95.8" x2="-92.38" y2="-110" width="0" layer="19" extent="1-1"/>
-<wire x1="37.62" y1="20" x2="-101.975" y2="-95.8" width="0" layer="19" extent="1-1"/>
-<wire x1="-61.9" y1="-82.125" x2="37.62" y2="20" width="0" layer="19" extent="1-1"/>
+<wire x1="-61.9" y1="-82.125" x2="-92.38" y2="-110" width="0" layer="19" extent="1-1"/>
 <wire x1="-61.9" y1="-76.125" x2="-61.9" y2="-82.125" width="0" layer="19" extent="1-1"/>
 <wire x1="-27.4665" y1="4.87113125" x2="-61.9" y2="-76.125" width="0" layer="19" extent="1-1"/>
 <wire x1="20.5" y1="14" x2="-27.4665" y2="4.87113125" width="0" layer="19" extent="1-16"/>
+<wire x1="37.62" y1="20" x2="20.5" y2="14" width="0" layer="19" extent="1-16"/>
 </signal>
 <signal name="CS_RFM">
@@
 <contactref element="U$6" pad="3"/>
 <contactref element="U$6" pad="1"/>
-<wire x1="32.54" y1="20" x2="30" y2="20" width="0" layer="19" extent="1-1"/>
+<wire x1="30" y1="20" x2="32.54" y2="20" width="0" layer="19" extent="1-1"/>
 </signal>
 <signal name="N$8">
 <contactref element="U$6" pad="2"/>
 <contactref element="U$6" pad="4"/>
-<wire x1="33.81" y1="20" x2="31.27" y2="20" width="0" layer="19" extent="1-1"/>
+<wire x1="31.27" y1="20" x2="33.81" y2="20" width="0" layer="19" extent="1-1"/>
 </signal>
 <signal name="N$9">
 <contactref element="U$6" pad="14"/>
 <contactref element="U$6" pad="12"/>
-<wire x1="32.54" y1="29.2" x2="30" y2="29.2" width="0" layer="19" extent="1-1"/>
+<wire x1="30" y1="29.2" x2="32.54" y2="29.2" width="0" layer="19" extent="1-1"/>
 </signal>
 <signal name="N$10">

Commit message: Partiall routed
Parts:
- removed J5: I2C2, SparkFun-Connectors:1X04
- added C16, C17, C18: 100nf, Seeed-Capacitor:C0603
- IC2: value W25Q32BVWSON8_6X5 -> (none)
- J4: value I2C1 -> GPS
- J6: value GPS -> I2C
- moved J7 341.0 mm to (67.0, 30.0)
- moved K1 320.4 mm to (73.0, 14.0)
- moved J6 276.5 mm to (38.0, 2.00)
- moved C14 257.7 mm to (34.0, 27.0)
- moved IC2 249.2 mm to (44.0, 30.0), turned to 270 degrees
- moved C13 240.3 mm to (27.0, 20.0), turned to 270 degrees
- moved R8 239.9 mm to (29.0, 10.0)
- moved J4 232.8 mm to (14.0, 2.00)
- moved C15 231.5 mm to (9.00, 10.0), turned to 270 degrees
- moved R7 213.2 mm to (8.00, 20.0), turned to 270 degrees
- moved U$7 204.0 mm to (53.0, 25.0)
- moved J3 193.1 mm to (2.00, 15.0), turned to 90 degrees
- moved R6 192.5 mm to (20.0, 22.0), turned to 270 degrees
- moved J2 190.4 mm to (29.0, 4.00), turned to 90 degrees
- moved R5 187.7 mm to (20.0, 20.0), turned to 270 degrees
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Connections:
- net N$6 renamed ANT
- removed net N$18: R8.1, U1.13
- new net BTN: K1.1, U1.25
- new net CS_FLASH: IC2.1, U1.36
- new net CS_SD: J7.2, U1.39
- new net MRST: J4.2, U1.20
- new net MTSR: J4.1, U1.21
- new net RESET: J2.3, R8.1, U1.13
- net CS_5525_1: now also U1.31
- net CS_5525_2: now also U1.27
- net CS_BMP: now also U1.1
- net GND: now also C16.1, C17.1, C18.1, IC2.4, J2.4, J4.3, J6.1, J7.6, J7.G1, J7.G2, J7.G3, J7.G4, K1.2, K1.3
- net LED_B: now also U1.41
- net LED_G: now also U1.40
- net MISO: now also IC2.2, J2.1, J7.7
- net MOSI: now also IC2.5, J2.5, J7.3
- net RC_IN: now also U1.28
- net RFM_D1: now also U1.29
- net RFM_D2: now also U1.30
- net SCK: now also IC2.6, J2.2, J7.5
- net SCL: now also J6.4
- net SDA: now also J6.3
- net VCC: now also C16.2, C17.2, C18.2, IC2.3, IC2.7, IC2.8, J2.6, J4.4, J6.2, J7.4
Routing:
- net SCK: track 0.00 -> 97.7 mm, vias 0 -> 2
- net MISO: track 0.00 -> 85.0 mm, vias 0 -> 4
- net MOSI: track 0.00 -> 83.2 mm, vias 0 -> 3
- net VCC: track 0.00 -> 80.1 mm, vias 0 -> 1
- net GND: track 0.00 -> 69.4 mm
- net V_USB: track 0.00 -> 43.3 mm
- net D+: track 0.00 -> 29.5 mm, vias 0 -> 2
- net D-: track 0.00 -> 29.0 mm, vias 0 -> 2
- net SCL: track 0.00 -> 19.3 mm, vias 0 -> 1
- net SDA: track 0.00 -> 17.6 mm
- net N$5: track 0.00 -> 13.5 mm
- net RESET: track 0.00 -> 9.08 mm
- net CS_BMP: track 0.00 -> 8.22 mm, vias 0 -> 2
- net N$2: track 0.00 -> 7.88 mm
- net N$16: track 0.00 -> 7.27 mm
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Other:
- board size 61 x 34 mm -> 80 x 40 mm

Commit message: partially routed
Parts:
- removed J4: GPS, SparkFun-Connectors:1X04
- removed R7: 2.2K, Seeed-Resistor:R0603
- added Q1, Q2: CJ2302, Seeed-Transistor:SOT-23
- added R10, R9: 2.2K, Seeed-Resistor:R0603
- added R11: 47K, Seeed-Resistor:R0603
- J3: value 455-1750-1-ND -> (none)
- moved U2 50.2 mm to (68.0, 11.0), turned to 270 degrees
- moved C2 15.5 mm to (52.3, 35.9), turned to 90 degrees
- moved J6 14.0 mm to (24.0, 2.00)
- moved J2 11.0 mm to (40.0, 3.00)
- moved C13 7.07 mm to (20.0, 21.0), turned to 90 degrees
- moved D1 5.00 mm to (8.52, 12.6)
- moved C14 5.00 mm to (31.0, 31.0)
- moved U3 4.12 mm to (16.9, 9.56)
- moved C1 4.00 mm to (16.0, 3.00)
- moved C5 4.00 mm to (19.0, 3.00)
- moved C12 3.61 mm to (39.0, 11.0)
- moved C6 3.61 mm to (37.0, 11.0)
- moved U1 3.61 mm to (32.9, 18.4)
- moved U4 3.61 mm to (43.0, 11.0)
- moved U$6 3.16 mm to (52.0, 4.00)
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Connections:
- removed net MRST: J4.2, U1.20
- removed net MTSR: J4.1, U1.21
- removed net N$17: J3.3, R7.2
- new net N$6: Q2.3, R10.1
- new net RX_INV: Q1.3, R9.1, U1.20
- new net TX_INV: Q2.1, U1.21
- net CS_BMP: now also U1.40; no longer U1.1
- net GND: now also Q1.2, Q2.2; no longer J4.3
- net LED_G: now also U1.1; no longer U1.40
- net RC_IN: now also J3.3, Q1.1, R10.2, R11.1; no longer R7.1, U1.28
- net VCC: now also R11.2, R9.2; no longer J4.4
Routing:
- net SCK: track 97.7 -> 47.4 mm, vias 2 -> 0
- net RX_INV: track 0.00 -> 38.7 mm, vias 0 -> 2
- net MISO: track 85.0 -> 46.3 mm, vias 4 -> 2
- net MOSI: track 83.2 -> 44.7 mm, vias 3 -> 0
- net GND: track 69.4 -> 38.5 mm
- net TX_INV: track 0.00 -> 29.8 mm, vias 0 -> 2
- net SDA: track 17.6 -> 36.0 mm, vias 0 -> 4
- net SCL: track 19.3 -> 34.5 mm, vias 1 -> 4
- net RESET: track 9.08 -> 23.7 mm, vias 0 -> 1
- net RC_IN: track 0.00 -> 10.8 mm
- net LED_G: track 0.00 -> 10.3 mm
- net CS_BMP: track 8.22 -> 0.00 mm, vias 2 -> 0
- net N$13: track 6.94 -> 0.00 mm
- net N$12: track 6.54 -> 0.00 mm
- net N$11: track 6.54 -> 0.00 mm
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Other:
- board size 80 x 40 mm -> 78 x 40 mm

Commit message: done routing!
Parts:
- moved C14 5.10 mm to (30.0, 26.0), turned to 90 degrees
- moved C3 3.16 mm to (53.0, 16.0)
- moved C7 3.00 mm to (57.0, 16.0)
Connections:
- net BTN: now also U1.28; no longer U1.25
- net CS_5525_1: now also U1.29; no longer U1.31
- net CS_5525_2: now also U1.32; no longer U1.27
- net CS_RFM: now also U1.30; no longer U1.8
- net CS_SD: now also U1.31; no longer U1.39
- net RFM_D0: now also U1.27; no longer U1.32
- net RFM_D1: now also U1.26; no longer U1.29
- net RFM_D2: now also U1.25; no longer U1.30
Routing:
- net VCC: track 80.5 -> 282.3 mm, vias 4 -> 8
- net SCK: track 47.4 -> 188.9 mm, vias 0 -> 6
- net MISO: track 46.3 -> 182.7 mm, vias 2 -> 8
- net MOSI: track 44.7 -> 178.6 mm, vias 0 -> 9
- net GND: track 38.5 -> 89.2 mm, vias 0 -> 61
- net CS_RFM: track 0.00 -> 40.8 mm, vias 0 -> 3
- net BTN: track 0.00 -> 40.4 mm, vias 0 -> 2
- net CS_SD: track 0.00 -> 39.7 mm, vias 0 -> 4
- net RFM_D0: track 0.00 -> 35.4 mm, vias 0 -> 1
- net CS_5611_1: track 0.00 -> 34.1 mm, vias 0 -> 4
- net RFM_D1: track 0.00 -> 33.7 mm, vias 0 -> 1
- net CS_5525_2: track 0.00 -> 33.1 mm, vias 0 -> 2
- net RFM_D2: track 0.00 -> 31.6 mm, vias 0 -> 1
- net CS_5525_1: track 0.00 -> 30.0 mm
- net SDA: track 36.0 -> 61.3 mm, vias 4 -> 6
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- added copper zone on layer 1, net GND
- added copper zone on layer 16, net GND

Commit message: Added silkscreen
Parts:
- moved J1 0.30 mm to (1.52, 6.25)
Other:
- board text added: "BMP280"
- board text added: "MS5525_1"
- board text added: "MS5525_2"
- board text added: "MS5611_1"
- board text added: "MS5611_2"
- board text added: "MS5637"
- board text added: "May the lift be with you"
- board text added: "RVario6 Designed by Patrick Grady the Great Feb 2019, when I should've been working on homework instead :/ Featuring too many pressure sensors and an IMU!!!"
- board text added: "S.PORT VIN GND"
- board text added: "SCL SDA VCC GND"
Changed lines of the file:
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@@
 <layer number="21" name="tPlace" color="7" fill="1" visible="yes" active="yes"/>
 <layer number="22" name="bPlace" color="7" fill="1" visible="yes" active="yes"/>
-<layer number="23" name="tOrigins" color="15" fill="1" visible="yes" active="yes"/>
-<layer number="24" name="bOrigins" color="15" fill="1" visible="yes" active="yes"/>
-<layer number="25" name="tNames" color="7" fill="1" visible="no" active="yes"/>
-<layer number="26" name="bNames" color="7" fill="1" visible="no" active="yes"/>
+<layer number="23" name="tOrigins" color="15" fill="1" visible="no" active="yes"/>
+<layer number="24" name="bOrigins" color="15" fill="1" visible="no" active="yes"/>
+<layer number="25" name="tNames" color="7" fill="1" visible="yes" active="yes"/>
+<layer number="26" name="bNames" color="7" fill="1" visible="yes" active="yes"/>
 <layer number="27" name="tValues" color="7" fill="1" visible="no" active="yes"/>
 <layer number="28" name="bValues" color="7" fill="1" visible="no" active="yes"/>
-<layer number="29" name="tStop" color="7" fill="3" visible="no" active="yes"/>
-<layer number="30" name="bStop" color="7" fill="6" visible="no" active="yes"/>
+<layer number="29" name="tStop" color="7" fill="3" visible="yes" active="yes"/>
+<layer number="30" name="bStop" color="7" fill="6" visible="yes" active="yes"/>
 <layer number="31" name="tCream" color="7" fill="4" visible="no" active="yes"/>
 <layer number="32" name="bCream" color="7" fill="5" visible="no" active="yes"/>
@@
 <wire x1="78" y1="40" x2="0" y2="40" width="0" layer="20"/>
 <wire x1="0" y1="40" x2="0" y2="0" width="0" layer="20"/>
+<text x="23.3" y="3.5" size="1.6764" layer="22" rot="MR90">SCL
+SDA
+VCC
+GND</text>
+<text x="13" y="21" size="1.6764" layer="22" rot="MR180" align="bottom-right">S.PORT
+VIN
+GND</text>
+<text x="13" y="36" size="1.27" layer="21" align="bottom-right">MS5611_1</text>
+<text x="24.7" y="38.1" size="1.27" layer="21" align="bottom-right">MS5611_2</text>
+<text x="26.5" y="24.9" size="1.27" layer="21" align="bottom-right">BMP280</text>
+<text x="39.1" y="38.6" size="1.27" layer="21" rot="R90" align="bottom-right">MS5637</text>
+<text x="54.4" y="38.2" size="1.27" layer="21" rot="R180" align="bottom-right">MS5525_2</text>
+<text x="59.9" y="0.9" size="1.27" layer="21" align="bottom-right">MS5525_1</text>
+<text x="73" y="22" size="1.27" layer="22" rot="MR0">RVario6
+Designed by Patrick Grady the Great
+Feb 2019, when I should've been
+working on homework instead :/
+Featuring too many pressure sensors
+and an IMU!!!</text>
+<text x="63.6" y="6.8" size="1.27" layer="21">May the lift
+be with you</text>
 </plain>
 <attributes>
@@
 </class>
 </classes>
-<designrules name="PATRICK-2lyr *">
+<designrules name="PATRICK-2lyr">
 <description language="en">&lt;b&gt;OSH Park Design Rules&lt;/b&gt;
 &lt;p&gt;
@@
 <param name="mdSmdStop" value="0mil"/>
 <param name="msWidth" value="6mil"/>
-<param name="msDrill" value="15mil"/>
+<param name="msDrill" value="10mil"/>
 <param name="msMicroVia" value="10mil"/>
 <param name="msBlindViaRatio" value="0.5"/>
@@
 <attribute name="PROD_ID" value="IC-10828" x="32.87" y="18.35" size="1.778" layer="27" display="off"/>
 </element>
-<element name="J1" library="Seeed-Connector" package="MICRO-USB5+6P-SMD-0.65-AB" value="ZX62-B-5PA" x="1.82" y="6.25" rot="R270">
-<attribute name="MPN" value="ZX62-B-5PA" x="1.82" y="6.25" size="1.778" layer="27" rot="R270" display="off"/>
+<element name="J1" library="Seeed-Connector" package="MICRO-USB5+6P-SMD-0.65-AB" value="ZX62-B-5PA" x="1.52" y="6.25" rot="R270">
+<attribute name="MPN" value="ZX62-B-5PA" x="1.52" y="6.25" size="1.778" layer="27" rot="R270" display="off"/>
 </element>
 <element name="Y1" library="Seeed-Crystal Oscillator" package="X3-SMD-3.6X1.3X0.8MM" value="8MHZ" x="32.95" y="11.02" rot="R270"/>
@@
 <contactref element="Q2" pad="2"/>
 <contactref element="Q1" pad="2"/>
-<wire x1="1.82" y1="2.625" x2="1.82" y2="4" width="0.1524" layer="1"/>
-<wire x1="1.82" y1="4" x2="1.82" y2="5.05" width="0.1524" layer="1"/>
-<wire x1="1.82" y1="5.05" x2="1.82" y2="7.45" width="0.1524" layer="1"/>
-<wire x1="1.82" y1="7.45" x2="1.82" y2="9.875" width="0.1524" layer="1"/>
-<wire x1="4.55" y1="8.675" x2="3.02" y2="8.675" width="0.1524" layer="1"/>
-<wire x1="3.02" y1="8.675" x2="1.82" y2="9.875" width="0.1524" layer="1"/>
-<wire x1="4.695" y1="4.95" x2="4.695" y2="3.97" width="0.1524" layer="1"/>
-<wire x1="4.695" y1="3.97" x2="4.55" y2="3.825" width="0.1524" layer="1"/>
-<wire x1="4.55" y1="3.825" x2="4.375" y2="4" width="0.1524" layer="1"/>
+<wire x1="1.52" y1="2.625" x2="1.82" y2="4" width="0.1524" layer="1"/>
+<wire x1="1.82" y1="4" x2="1.52" y2="5.05" width="0.1524" layer="1"/>
+<wire x1="1.52" y1="5.05" x2="1.52" y2="7.45" width="0.1524" layer="1"/>
+<wire x1="1.52" y1="7.45" x2="1.52" y2="9.875" width="0.1524" layer="1"/>
+<wire x1="4.25" y1="8.675" x2="3.02" y2="8.675" width="0.1524" layer="1"/>
+<wire x1="3.02" y1="8.675" x2="1.52" y2="9.875" width="0.1524" layer="1"/>
+<wire x1="4.395" y1="4.95" x2="4.695" y2="3.97" width="0.1524" layer="1"/>
+<wire x1="4.695" y1="3.97" x2="4.25" y2="3.825" width="0.1524" layer="1"/>
+<wire x1="4.25" y1="3.825" x2="4.375" y2="4" width="0.1524" layer="1"/>
 <wire x1="4.375" y1="4" x2="1.82" y2="4" width="0.1524" layer="1"/>
 <wire x1="2" y1="15" x2="1.82" y2="14.82" width="0.1524" layer="1"/>
-<wire x1="1.82" y1="14.82" x2="1.82" y2="9.875" width="0.1524" layer="1"/>
+<wire x1="1.82" y1="14.82" x2="1.52" y2="9.875" width="0.1524" layer="1"/>
 <wire x1="37" y1="10.238" x2="39" y2="10.238" width="0.1524" layer="1"/>
 <wire x1="42.238" y1="7.7" x2="42.8" y2="8.262" width="0.1524" layer="1"/>
@@
 <via x="61.5" y="13.8" extent="1-16" drill="0.6"/>
 <via x="50" y="16" extent="1-16" drill="0.6"/>
-<wire x1="43.6" y1="12.5" x2="43.6" y2="11.8" width="0.1524" layer="1"/>
-<wire x1="43.6" y1="11.8" x2="43.8496125" y2="11.8" width="0.1524" layer="1"/>
-<wire x1="43.8496125" y1="11.8" x2="44.0496125" y2="12" width="0.1524" layer="1"/>
-<wire x1="44.0496125" y1="12" x2="44.5" y2="12" width="0.1524" layer="1"/>
+<wire x1="43.6" y1="11.8" x2="43.6" y2="11.9" width="0.1524" layer="1"/>
+<wire x1="43.6" y1="11.9" x2="43.6" y2="12.5" width="0.1524" layer="1"/>
+<wire x1="43.8496125" y1="11.8" x2="43.6" y2="11.8" width="0.1524" layer="1"/>
 <via x="43" y="15" extent="1-16" drill="0.6"/>
 <via x="46" y="12" extent="1-16" drill="0.6"/>
@@
 <via x="77" y="14" extent="1-16" drill="0.6"/>
 <via x="73" y="14" extent="1-16" drill="0.6"/>
+<wire x1="44.5" y1="12" x2="44.4286" y2="11.9286" width="0.1524" layer="1"/>
+<wire x1="44.4286" y1="11.9286" x2="44.1346" y2="11.9286" width="0.1524" layer="1"/>
+<wire x1="44.1346" y1="11.9286" x2="44.106" y2="11.9" width="0.1524" layer="1"/>
+<wire x1="44.106" y1="11.9" x2="43.6" y2="11.9" width="0.1524" layer="1"/>
 </signal>
 <signal name="N$3">
 <contactref element="J1" pad="2"/>
 <contactref element="R1" pad="1"/>
-<wire x1="4.695" y1="6.9" x2="6.1" y2="6.9" width="0.1524" layer="1"/>
+<wire x1="4.395" y1="6.9" x2="6.1" y2="6.9" width="0.1524" layer="1"/>
 <wire x1="6.1" y1="6.9" x2="7" y2="6" width="0.1524" layer="1"/>
 <wire x1="7" y1="6" x2="8.15" y2="6" width="0.1524" layer="1"/>
@@
 <contactref element="J1" pad="3"/>
 <contactref element="R2" pad="1"/>
-<wire x1="4.695" y1="6.25" x2="5.9" y2="6.25" width="0.1524" layer="1"/>
+<wire x1="4.395" y1="6.25" x2="5.9" y2="6.25" width="0.1524" layer="1"/>
 <wire x1="5.9" y1="6.25" x2="8.15" y2="4" width="0.1524" layer="1"/>
 </signal>
@@
 <contactref element="U1" pad="7"/>
 <contactref element="C15" pad="2"/>
-<wire x1="4.695" y1="7.55" x2="7.661" y2="7.55" width="0.254" layer="1"/>
+<wire x1="4.395" y1="7.55" x2="7.661" y2="7.55" width="0.254" layer="1"/>
 <wire x1="7.661" y1="7.55" x2="8.0555" y2="7.9445" width="0.254" layer="1"/>
 <wire x1="8.0555" y1="7.9445" x2="8.111" y2="8" width="0.254" layer="1"/>
@@
 </drawing>
 <compatibility>
+<note version="6.3" minversion="6.2.2" severity="warning">
+Since Version 6.2.2 text objects can contain more than one line,
+which will not be processed correctly with this version.
+</note>
 <note version="8.3" severity="warning">
 Since Version 8.3, EAGLE supports URNs for individual library

Commit message: SEEED SUBMIT!!!!!
Parts:
- R1, R2: value 22 -> 22R; device SparkFun-Resistors:0603 -> Seeed-Resistor:R0603
- turned R1 to 90 degrees
- turned R2 to 90 degrees
- renumbered U$3 to S4, U$4 to S5, U$5 to S3, U$6 to S2, U$7 to S1
