File: RVario6/main.sch (EAGLE design)
At the start: 54 parts, among them IC1 BMP280, IC2 W25Q32BVWSON8_6X5, J1 ZX62-B-5PA, J2 2x3p-2.54, J6 I2C, J7 MICROSD-9P, Q1 CJ2302, Q2 CJ2302, U1 32U4, U2 433MHz, U3 CJT1117-3.3-SOT223, Y1 8MHZ

Commit message: done routing!
Connections:
- net BTN: now also U1.PB4(ADC11); no longer U1.PD4(ADC8)
- net CS_5525_1: now also U1.PB5(ADC12); no longer U1.PC6
- net CS_5525_2: now also U1.PC7; no longer U1.PD7(ADC10)
- net CS_RFM: now also U1.PB6(ADC13); no longer U1.PB0(SS)
- net CS_SD: now also U1.PC6; no longer U1.PF4(ADC4)
- net RFM_D0: now also U1.PD7(ADC10); no longer U1.PC7
- net RFM_D1: now also U1.PD6(ADC9); no longer U1.PB5(ADC12)
- net RFM_D2: now also U1.PD4(ADC8); no longer U1.PB6(ADC13)
Changed lines of the file:
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@@
 </segment>
 <segment>
-<pinref part="U1" gate="U1" pin="PB0(SS)"/>
-<wire x1="124.46" y1="53.34" x2="134.62" y2="53.34" width="0.1524" layer="91"/>
-<label x="127" y="53.34" size="1.778" layer="95"/>
+<pinref part="U1" gate="U1" pin="PB6(ADC13)"/>
+<wire x1="124.46" y1="63.5" x2="139.7" y2="63.5" width="0.1524" layer="91"/>
+<label x="129.54" y="63.5" size="1.778" layer="95"/>
 </segment>
 </net>
@@
 </segment>
 <segment>
-<pinref part="U1" gate="U1" pin="PC7"/>
-<wire x1="124.46" y1="55.88" x2="134.62" y2="55.88" width="0.1524" layer="91"/>
-<label x="127" y="55.88" size="1.778" layer="95"/>
+<pinref part="U1" gate="U1" pin="PD7(ADC10)"/>
+<wire x1="124.46" y1="73.66" x2="139.7" y2="73.66" width="0.1524" layer="91"/>
+<label x="129.54" y="73.66" size="1.778" layer="95"/>
 </segment>
 </net>
@@
 </segment>
 <segment>
-<pinref part="U1" gate="U1" pin="PD7(ADC10)"/>
-<wire x1="124.46" y1="73.66" x2="139.7" y2="73.66" width="0.1524" layer="91"/>
-<label x="129.54" y="73.66" size="1.778" layer="95"/>
+<pinref part="U1" gate="U1" pin="PC7"/>
+<wire x1="124.46" y1="55.88" x2="139.7" y2="55.88" width="0.1524" layer="91"/>
+<label x="129.54" y="55.88" size="1.778" layer="95"/>
 </segment>
 </net>
@@
 </segment>
 <segment>
-<pinref part="U1" gate="U1" pin="PC6"/>
-<wire x1="124.46" y1="76.2" x2="139.7" y2="76.2" width="0.1524" layer="91"/>
-<label x="129.54" y="76.2" size="1.778" layer="95"/>
+<pinref part="U1" gate="U1" pin="PB5(ADC12)"/>
+<wire x1="124.46" y1="66.04" x2="139.7" y2="66.04" width="0.1524" layer="91"/>
+<label x="129.54" y="66.04" size="1.778" layer="95"/>
 </segment>
 </net>
@@
 </segment>
 <segment>
-<pinref part="U1" gate="U1" pin="PB5(ADC12)"/>
-<wire x1="124.46" y1="66.04" x2="139.7" y2="66.04" width="0.1524" layer="91"/>
-<label x="129.54" y="66.04" size="1.778" layer="95"/>
+<pinref part="U1" gate="U1" pin="PD6(ADC9)"/>
+<wire x1="124.46" y1="58.42" x2="139.7" y2="58.42" width="0.1524" layer="91"/>
+<label x="129.54" y="58.42" size="1.778" layer="95"/>
 </segment>
 </net>
@@
 </segment>
 <segment>
-<pinref part="U1" gate="U1" pin="PB6(ADC13)"/>
-<wire x1="124.46" y1="63.5" x2="139.7" y2="63.5" width="0.1524" layer="91"/>
-<label x="129.54" y="63.5" size="1.778" layer="95"/>
+<pinref part="U1" gate="U1" pin="PD4(ADC8)"/>
+<wire x1="124.46" y1="78.74" x2="139.7" y2="78.74" width="0.1524" layer="91"/>
+<label x="129.54" y="78.74" size="1.778" layer="95"/>
 </segment>
 </net>
@@
 </segment>
 <segment>
-<pinref part="U1" gate="U1" pin="PD4(ADC8)"/>
-<wire x1="124.46" y1="78.74" x2="139.7" y2="78.74" width="0.1524" layer="91"/>
-<label x="129.54" y="78.74" size="1.778" layer="95"/>
+<pinref part="U1" gate="U1" pin="PB4(ADC11)"/>
+<wire x1="124.46" y1="68.58" x2="139.7" y2="68.58" width="0.1524" layer="91"/>
+<label x="129.54" y="68.58" size="1.778" layer="95"/>
 </segment>
 </net>
@@
 </segment>
 <segment>
-<pinref part="U1" gate="U1" pin="PF4(ADC4)"/>
-<wire x1="124.46" y1="104.14" x2="139.7" y2="104.14" width="0.1524" layer="91"/>
-<label x="129.54" y="104.14" size="1.778" layer="95"/>
-</segment>
-</net>
+<pinref part="U1" gate="U1" pin="PC6"/>
+<wire x1="124.46" y1="76.2" x2="139.7" y2="76.2" width="0.1524" layer="91"/>
+<label x="129.54" y="76.2" size="1.778" layer="95"/>
+</segment>
+</net>

Commit message: SEEED SUBMIT!!!!!
Parts:
- R1, R2: value 22 -> 22R; device SparkFun-Resistors:RESISTOR0603 -> Seeed-Resistor:SMD-RES-22R-5%-1/10W(0603)
- renumbered U$3 to S4, U$4 to S5, U$5 to S3, U$6 to S2, U$7 to S1
