File: VarioBase/main.brd (EAGLE design)
At the start: 54 x 60 mm, 17 parts, among them J1 HEADER4VALULOK, J2 HEADER4VALULOK, J3 HEADER4VALULOK, J4 HEADER4VALULOK, J5 BT, J6 SD

Commit message: JLC submit
Parts:
- removed J4: HEADER4VALULOK, Custom_old:4PINVALULOK
- removed J5: BT, SparkFun-Connectors:1X04_NO_SILK
- removed J6: SD, SparkFun-Connectors:1X06_NO_SILK
- removed U$2: FUSE, Custom_old:AUTO_FUSE
- removed U$4: TEENSY_3.0_BASIC, Teensy3.0:TEENSY_3.0_BASIC
- added BT1: HC06, 2020:HC06
- added C1, C10, C11, C2, C3, C4, C5, C6, C7, C8, C9: 10uF, SparkFun-Capacitors:1206
- added C12, C14: 0.1uF, SparkFun-Capacitors:0603
- added S1: MS4525, 2020:DIP1270W53P254L990H762Q8B
- added S2: MS5611, Custom_old:MS5611
- added U1: (no value), SparkFun-IC-Power:SOT223
- added U2: (no value), SparkFun-IC-Power:V-REG_DPACK
- U$1: value PB -> TEENSY_3.5/3.6_BASIC; device Custom_old:8PINVALULOK -> Teensy356:TEENSY_3.5/3.6_BASIC
- moved JP4 40.5 mm to (21.0, 50.0)
- moved U$3 40.1 mm to (4.00, 60.0)
- moved U$1 25.1 mm to (39.4, 32.0), turned to 270 degrees
- moved R1 18.4 mm to (28.0, 38.0)
- moved J2 16.8 mm to (13.0, 19.0), turned to 180 degrees
- moved J3 16.5 mm to (26.0, 19.0), turned to 180 degrees
- moved R2 16.5 mm to (26.0, 38.0)
- moved JP1 14.4 mm to (9.00, 24.0)
- moved J1 11.8 mm to (8.80, 9.00), flipped to the bottom, turned to 180 degrees
- moved JP3 11.3 mm to (24.0, 24.0)
- moved JP2 8.94 mm to (14.0, 24.0)
Connections:
- removed net 3.3V: U$4.3.3V, U$4.3.3V1
- removed net CS_PITOT: B1.A4, U$1.8
- removed net CS_SD: B1.A5, J6.5
- removed net CS_STATIC: B1.A3, U$1.6
- removed net CS_TE: B1.A2, U$1.7
- removed net N$5: U$2.1A, U$2.1B, U$3.1
- removed net RES_CS_IMU: B1.D10
- removed net RES_PSEL0: B1.D9
- removed net RES_PSEL1: B1.D8
- removed net RES_RSTIMU: B1.D4
- removed net UART_MISO: B1.RX, J3.4, J4.4, J5.3
- removed net UART_MOSI: B1.TX, J3.3, J4.3, J5.4
- removed net VBAT: U$4.VBAT
- new net 33_CLEAN: C10.1, C12.1, C9.1, JP4.3, S2.1, S2.2, U1.2
- new net 4525_INT: S1.5, U$1.2
- new net BT_UART_MISO: BT1.3, U$1.9/CS
- new net BT_UART_MOSI: BT1.4, U$1.10/CS
- new net CS_IMU: B1.D10, U$1.16/A2
- new net IMU_RST: B1.D4, U$1.37/A18
- new net IMU_UART_CTS: B1.D3, U$1.36/A17
- new net IMU_UART_MISO: B1.RX, U$1.34/A15
- new net IMU_UART_MOSI: B1.TX, U$1.33/A14
- new net IMU_UART_RTS: B1.D2, U$1.35/A16
- new net PSEL0: B1.D9, U$1.15/A1
- new net PSEL1: B1.D8, U$1.A22/DAC1
- new net RTK_UART_MISO: J3.4, U$1.31/A12
- new net RTK_UART_MOSI: J3.3, U$1.32/A13
- net 5V: now also BT1.1, C5.1, C6.1, C7.1, C8.1, JP4.1, U$1.VIN, U1.3, U2.3; no longer J5.1, JP4.3, U$1.2, U$4.VIN
- net GND: now also BT1.2, C1.2, C10.2, C11.2, C12.2, C14.2, C2.2, C3.2, C4.2, C5.2, C6.2, C7.2, C8.2, C9.2, S1.1, S2.3, S2.4, S2.5, U$1.AGND, U$1.GND, U$1.GND2, U1.1, U2.1; no longer J4.2, J5.2, J6.1, U$1.1, U$4.AGND, U$4.GND, U$4.GND1
- net MISO: now also U$1.12/MISO; no longer J6.2, U$1.3
- net MOSI: now also U$1.11/MOSI; no longer J6.4, U$1.4
- net N$4: now also C11.1, C14.1, S1.2; no longer J4.1
- net SCL: now also S1.4, S2.8, U$1.19/A5/SCL
- net SCLK: now also U$1.14/A0; no longer J6.3, U$1.5
- net SDA: now also S1.3, S2.7, U$1.18/A4/SDA
- net VCC: now also B1.IOREF, U$1.3V3, U$1.3V3_LO; no longer J6.6, JP4.1
- net VIN: now also C1.1, C2.1, C3.1, C4.1, U$3.1, U2.4; no longer B1.VIN, U$2.2A, U$2.2B
Routing:
- net CS_STATIC: track 63.0 -> 0.00 mm, vias 1 -> 0
- net CS_PITOT: track 58.6 -> 0.00 mm
- net UART_MISO: track 51.1 -> 0.00 mm, vias 1 -> 0
- net CS_SD: track 50.6 -> 0.00 mm, vias 2 -> 0
- net CS_TE: track 49.2 -> 0.00 mm, vias 1 -> 0
- net GND: track 2.54 -> 46.4 mm, vias 0 -> 15
- net MOSI: track 64.3 -> 21.0 mm, vias 1 -> 0
- net SCLK: track 59.3 -> 17.5 mm, vias 2 -> 0
- net UART_MOSI: track 38.4 -> 0.00 mm
- net MISO: track 56.7 -> 24.5 mm, vias 2 -> 1
- net 33_CLEAN: track 0.00 -> 29.4 mm, vias 0 -> 2
- net SCL: track 77.8 -> 104.4 mm, vias 5 -> 8
- net VIN: track 40.6 -> 20.1 mm, vias 1 -> 0
- net RTK_UART_MISO: track 0.00 -> 20.2 mm
- net SDA: track 84.1 -> 103.2 mm, vias 4 -> 6
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- added copper zone on layer 1, net GND
Other:
- board size 54 x 60 mm -> 53 x 63 mm
- board text removed: "+5 GND"
- board text removed: "3.3"
- board text removed: "3.3/5"
- board text removed: "5v"
- board text removed: "Bluetooth"
- board text removed: "CS"
- board text removed: "CS_PIT CS_TE"
- board text removed: "CS_STAT SCLK"
- board text removed: "FUSE"
- board text removed: "GND"
- board text removed: "I2C"
- board text removed: "MISO"
- board text removed: "MOSI"
- board text removed: "MOSI MISO"
- board text removed: "Micro SD"
- board text removed: "SCL SDA"
- board text removed: "SCLK"
- board text removed: "SPI Pressure"
- board text removed: "UART"
- board text removed: "UART_MISO"
- board text removed: "UART_MOSI"
- board text removed: "UMOSI UMISO"
- board text removed: "VCC GND"
- board text removed: "VIN"
