File: VarioBase/main.sch (EAGLE design)
At the start: 17 parts, among them J1 HEADER4VALULOK, J2 HEADER4VALULOK, J3 HEADER4VALULOK, J4 HEADER4VALULOK, J5 BT, J6 SD

Commit message: JLC submit
Parts:
- removed J4: HEADER4VALULOK, Custom_old:HEADER4VALULOK
- removed J5: BT, SparkFun-Connectors:CONN_041X04_NO_SILK
- removed J6: SD, SparkFun-Connectors:CONN_06NO_SILK_NO_POP
- removed U$2: FUSE, Custom_old:FUSE
- removed U$4: TEENSY_3.0_BASIC, Teensy3.0:TEENSY_3.0_BASIC
- added BT1: HC06, 2020:HC06
- added C1, C10, C11, C2, C3, C4, C5, C6, C7, C8, C9: 10uF, SparkFun-Capacitors:10UF-1206-6.3V-20%
- added C12, C14: 0.1uF, SparkFun-Capacitors:0.1UF-0603-25V-5%
- added S1: MS4525, 2020:MS4525MS4525DO
- added S2: MS5611, Custom_old:MS5611
- added U1: V_REG_317SMD, SparkFun-IC-Power:V_REG_317SMD
- added U2: V_REG_317DPACK, SparkFun-IC-Power:V_REG_317DPACK
- U$1: value PB -> TEENSY_3.5/3.6_BASIC; device Custom_old:HEADER8 -> Teensy356:TEENSY_3.5/3.6_BASIC
Connections:
- removed net 3.3V: U$4.3.3V
- removed net CS_PITOT: B1.A4, U$1.8
- removed net CS_SD: B1.A5, J6.5
- removed net CS_STATIC: B1.A3, U$1.6
- removed net CS_TE: B1.A2, U$1.7
- removed net N$5: U$2.1, U$3.1
- removed net RES_CS_IMU: B1.*D10
- removed net RES_PSEL0: B1.*D9
- removed net RES_PSEL1: B1.D8
- removed net RES_RSTIMU: B1.D4
- removed net UART_MISO: B1.RX, J3.4, J4.4, J5.3
- removed net UART_MOSI: B1.TX, J3.3, J4.3, J5.4
- new net 33_CLEAN: C10.1, C12.1, C9.1, JP4.3, S2.PS, S2.VDD, U1.OUT
- new net 4525_INT: S1.INT, U$1.2
- new net BT_UART_MISO: BT1.UART_MISO, U$1.9/CS
- new net BT_UART_MOSI: BT1.UART_MOSI, U$1.10/CS
- new net CS_IMU: B1.*D10, U$1.16/A2
- new net IMU_RST: B1.D4, U$1.37/A18
- new net IMU_UART_CTS: B1.*D3, U$1.36/A17
- new net IMU_UART_MISO: B1.RX, U$1.34/A15
- new net IMU_UART_MOSI: B1.TX, U$1.33/A14
- new net IMU_UART_RTS: B1.D2, U$1.35/A16
- new net PSEL0: B1.*D9, U$1.15/A1
- new net PSEL1: B1.D8, U$1.A22/DAC1
- new net RTK_UART_MISO: J3.4, U$1.31/A12
- new net RTK_UART_MOSI: J3.3, U$1.32/A13
- net 5V: now also BT1.5V, C5.1, C6.1, C7.1, C8.1, JP4.1, U$1.VIN, U1.IN, U2.IN; no longer J5.1, JP4.3, U$1.2, U$4.VIN
- net GND: now also BT1.GND, C1.2, C10.2, C11.2, C12.2, C14.2, C2.2, C3.2, C4.2, C5.2, C6.2, C7.2, C8.2, C9.2, S1.GND, S2.CSB4, S2.CSB5, S2.GND, U$1.AGND, U$1.GND, U$1.GND2, U1.ADJ, U2.ADJ; no longer J4.2, J5.2, J6.1, U$1.1, U$4.AGND, U$4.GND
- net MISO: now also U$1.12/MISO; no longer J6.2, U$1.3
- net MOSI: now also U$1.11/MOSI; no longer J6.4, U$1.4
- net N$4: now also C11.1, C14.1, S1.V+; no longer J4.1
- net SCL: now also S1.SCL, S2.SCLK, U$1.19/A5/SCL
- net SCLK: now also U$1.14/A0; no longer J6.3, U$1.5
- net SDA: now also S1.SDA, S2.SDI/SDA, U$1.18/A4/SDA
- net VCC: now also B1.IOREF, U$1.3V3, U$1.3V3_LO; no longer J6.6, JP4.1
- net VIN: now also C1.1, C2.1, C3.1, C4.1, U$3.1, U2.OUT; no longer B1.VIN, U$2.2
Other:
- note added: "Accessories"
- note added: "Bluetooth"
- note added: "Pressure Board"
- note added: "RTK, stupid pinout"
- note removed: "PressureBoard"
- moved on the sheet: J3, JP3, JP4

Commit message: Added error note....
Other:
- note added: "OOOOPS BACKWARDS!!!!!!!!!!!!!! 5V flipped!!!!"
Changed lines of the file:
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@@
 <text x="167.64" y="101.6" size="1.778" layer="94">RTK, stupid pinout</text>
 <text x="205.74" y="101.6" size="1.778" layer="94">Bluetooth</text>
+<text x="58.42" y="137.16" size="1.778" layer="94">OOOOPS BACKWARDS!!!!!!!!!!!!!!
+5V flipped!!!!</text>
 </plain>
 <instances>
